File: hdw/rev_b/Audio_Optical_Trigger/Audio_Optical_Trigger.kicad_pcb (KiCad board)
At the start: 2 copper layers, 58.6 x 62.4 mm, 130 parts, among them J1001 Trigger Output, J201 +12VIN, J301 TX1, J302 RX1, J401 TX2, J402 RX2, J501 TX3, J502 RX3, J901 Group Select, Q201 IRF7404, U201 74LVC1G14, U202 TPS62130, U301 74LVC1G17, U401 74LVC1G17, U501 74LVC1G17, U601 74LVC1G38, U602 74LVC1G38, U603 74LVC1G38, U701 74LVC1G38, U702 74LVC1G38, U703 74LVC1G38, U801 74LVC1G38, U802 74LVC1G38, U803 74LVC1G38, U901 74LVC1G14, U902 74LVC1G14, U903 74LVC1G14

Commit message: routed rev b board, created BOM, generated gerbers
Parts:
- removed C602, C603, C801, C802, C803: 0.1uF, Capacitors_SMD:C_0603
- removed R601, R602, R603, R604, R605, R606, R607, R608, R609, R705, R706, R707, R708, R709, R801, R802, R803, R804, R805, R806, R807, R808, R809: 10k, Resistors_SMD:R_0603
- removed U601, U602, U603, U801, U802, U803: 74LVC1G38, TO_SOT_Packages_SMD:SOT-353_SC-70-5
- added C704: 0.1uF, Capacitors_SMD:C_0603, F.Cu at (150.5, 83.9)
- added C705: 0.1uF, Capacitors_SMD:C_0603, F.Cu at (150.5, 91.2)
- added D701: RED, LEDs:LED_0603, F.Cu at (153.7, 81.0)
- added D702: GREEN, LEDs:LED_0603, F.Cu at (153.7, 88.3)
- added J601: PICKIT3, Connector_PinHeader_2.54mm:PinHeader_1x06_P2.54mm_Vertical, F.Cu at (120.8, 110.3)
- C601: moved to B.Cu
- C702: value 0.1uF -> 10nF
- C703: value 0.1uF -> 1nF
- D302, D402, D502, D902, D903, D904: value MM5Z5V6 -> MM5Z3V6
- R701, R702: moved to F.Cu
- R703, R704: value 10k -> 2k; moved to F.Cu
- U701: value 74LVC1G38 -> PIC18F27K40T-I_ML; footprint TO_SOT_Packages_SMD:SOT-353_SC-70-5 -> Housings_DFN_QFN:QFN-28-1EP_6x6mm_Pitch0.65mm
- U702, U703: value 74LVC1G38 -> 74LVC1G14
- moved C601 36.8 mm to (124.7, 108.3), turned to 0 degrees
- moved REF*** 33.0 mm to (135.7, 99.6)
- moved R701 25.5 mm to (148.1, 82.8), turned to 90 degrees
- moved U702 21.9 mm to (150.5, 81.8)
- moved R704 18.8 mm to (153.5, 89.8), turned to 180 degrees
- moved C701 18.0 mm to (143.2, 98.8), turned to 0 degrees
- moved U701 15.1 mm to (142.2, 107.2), turned to 90 degrees
- moved C702 14.9 mm to (143.2, 100.2), turned to 0 degrees
- moved R703 14.5 mm to (153.5, 82.5), turned to 180 degrees
- moved R702 14.3 mm to (148.1, 90.5), turned to 270 degrees
- moved C703 14.3 mm to (143.2, 101.6), turned to 0 degrees
- moved G*** 11.8 mm to (154.7, 106.0)
- moved U703 10.9 mm to (150.5, 89.1)
- moved C206 2.49 mm to (138.4, 91.8)
- moved L201 2.49 mm to (143.8, 87.3)
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Connections:
- C201 pad 1: +5V -> +3V3
- C206 pad 1: +5V -> +3V3
- C207 pad 1: +5V -> +3V3
- C302 pad 1: +5V -> +3V3
- C402 pad 1: +5V -> +3V3
- C502 pad 1: +5V -> +3V3
- C601 pad 1: +5V -> +3V3
- C701 pad 1: +5V -> +3V3
- C702 pad 1: +5V -> +3V3
- C703 pad 1: +5V -> +3V3
- C904 pad 1: +5V -> +3V3
- C905 pad 1: +5V -> +3V3
- C906 pad 1: +5V -> +3V3
- D202 pad 2: +5V -> +3V3
- D301 pad 2: +5V -> +3V3
- D401 pad 2: +5V -> +3V3
- D501 pad 2: +5V -> +3V3
- D901 pad 6: (no net) -> Net-(D901-Pad6)
- J1001 pad 19: (no net) -> Net-(J1001-Pad19)
- J1001 pad 21: (no net) -> Net-(J1001-Pad21)
- J1001 pad 23: (no net) -> Net-(J1001-Pad23)
- J1001 pad 25: (no net) -> Net-(J1001-Pad25)
- J1001 pad 27: (no net) -> Net-(J1001-Pad27)
- J1001 pad 29: (no net) -> Net-(J1001-Pad29)
- J1001 pad 31: (no net) -> Net-(J1001-Pad31)
- J1001 pad 33: (no net) -> Net-(J1001-Pad33)
- J1001 pad 35: (no net) -> Net-(J1001-Pad35)
- J302 pad 1: +5V -> +3V3
- J402 pad 1: +5V -> +3V3
- J502 pad 1: +5V -> +3V3
- L201 pad 2: +5V -> +3V3
- R203 pad 1: +5V -> +3V3
- R203 pad 2: POS5_PGOOD -> POS3P3_PGOOD
- R206 pad 1: +5V -> +3V3
- R301 pad 1: +5V -> +3V3
- R303 pad 1: +5V -> +3V3
- R401 pad 1: +5V -> +3V3
- R403 pad 1: +5V -> +3V3
- R501 pad 1: +5V -> +3V3
- R503 pad 1: +5V -> +3V3
- R701 pad 1: Output_Group_Select_2 -> +3V3
- R701 pad 2: GND -> Reset_LED
- R702 pad 1: Output_Group_Select_2 -> Heartbeat_LED
- R703 pad 1: Output_Group_Select_2 -> Net-(D701-Pad1)
- R703 pad 2: GND -> Net-(R703-Pad2)
- R704 pad 1: Input_Channel_1 -> Net-(D702-Pad1)
- R704 pad 2: GND -> Net-(R704-Pad2)
- R904 pad 1: +5V -> +3V3
- R905 pad 1: +5V -> +3V3
- R906 pad 1: +5V -> +3V3
- TP203 pad 1: +5V -> +3V3
- U201 pad 2: POS5_PGOOD -> POS3P3_PGOOD
- U201 pad 5: +5V -> +3V3
- U202 pad 14: +5V -> +3V3
- U202 pad 4: POS5_PGOOD -> POS3P3_PGOOD
- U301 pad 5: +5V -> +3V3
- U401 pad 5: +5V -> +3V3
- U501 pad 5: +5V -> +3V3
- U701 pad 1: Output_Group_Select_2 -> Input_Channel_3
- U701 pad 2: Input_Channel_1 -> Output_Group_Select_1
- U701 pad 3: GND -> Output_Group_Select_2
- U701 pad 4: ~Output_Group_2_Channel_1 -> Output_Group_Select_3
- U701 pad 5: +5V -> GND
- U702 pad 1: Output_Group_Select_2 -> (no net)
- U702 pad 2: Input_Channel_2 -> Reset_LED
- U702 pad 4: ~Output_Group_2_Channel_2 -> Net-(R703-Pad2)
- U702 pad 5: +5V -> +3V3
- U703 pad 1: Output_Group_Select_2 -> (no net)
- U703 pad 2: Input_Channel_3 -> Heartbeat_LED
- U703 pad 4: ~Output_Group_2_Channel_3 -> Net-(R704-Pad2)
- U703 pad 5: +5V -> +3V3
- U901 pad 5: +5V -> +3V3
- U902 pad 5: +5V -> +3V3
- U903 pad 5: +5V -> +3V3
Routing:
- net POS3P3_PGOOD: track 0.00 -> 113.6 mm, vias 0 -> 5
- net Input_Channel_1: track 77.1 -> 16.9 mm, vias 6 -> 0
- net Input_Channel_2: track 64.0 -> 4.89 mm, vias 7 -> 0
- net POS5_PGOOD: track 56.7 -> 0.00 mm, vias 3 -> 0
- net +3V3: track 0.00 -> 55.3 mm, vias 0 -> 6
- net Input_Channel_3: track 51.0 -> 10.7 mm, vias 7 -> 0
- net Output_Group_Select_3: track 57.9 -> 19.9 mm, vias 7 -> 2
- net Output_Group_Select_1: track 64.7 -> 29.0 mm, vias 7 -> 2
- net Reset_LED: track 0.00 -> 29.8 mm, vias 0 -> 2
- net ~Output_Group_2_Channel_1: track 22.0 -> 47.9 mm
- net Output_Group_Select_2: track 49.4 -> 25.3 mm, vias 7 -> 2
- net ~Output_Group_2_Channel_2: track 20.9 -> 44.0 mm
- net Heartbeat_LED: track 0.00 -> 23.0 mm, vias 0 -> 2
- net ~MCLR: track 0.00 -> 22.5 mm
- net ~Output_Group_2_Channel_3: track 23.6 -> 43.8 mm
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- added copper zone on F.Cu, net +3V3
- removed copper zone on F.Cu, net +5V
Other:
- net class Default: via_dia 0.7 -> 0.4318; via_drill 0.3 -> 0.2
- net class Power: via_dia 0.7 -> 0.4318; via_drill 0.3 -> 0.2
- net class Signal: via_dia 0.7 -> 0.4318; via_drill 0.3 -> 0.2
- rule trace_min: 0.127 -> 0.0508
- rule via_min_drill: 0.3 -> 0.199898
- rule via_min_size: 0.6 -> 0.4
- board text added: "+3.3V"
- board text added: "+3.3V PGOOD"
- board text added: "HEART BEAT"
- board text added: "JLCJLCJLCJLC"
- board text added: "May 2020"
- board text added: "PICKIT3"
- board text added: "RESET"
- board text added: "Sparkfun MP3 Trigger Optical Interface REV B"
- board text removed: "+5V"
- board text removed: "+5V PGOOD"
- board text removed: "January 2019"
- board text removed: "Sparkfun MP3 Trigger Optical Interface"
